File: cpio-pcb/eagle-proj/cpio_v0.1/cpio_v0.1.brd (EAGLE design)
At the start: 100 x 80 mm, 95 parts

Commit message: rename brightness input. Now with gnd, signal, vcc
Parts:
- renumbered SENS_PH1 to SENS_BRIGHT
Changed lines of the file:
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@@
 <element name="SENS_I" library="cpio" package="SOT23-5" value="INA139" x="-30.48" y="59.69"/>
 <element name="SENS_PH" library="cpio" package="XH-A-3" value="XH-A-3" x="-60.96" y="46.99"/>
-<element name="SENS_PH1" library="cpio" package="XH-A-3" value="XH-A-3" x="-71.12" y="46.99"/>
+<element name="SENS_BRIGHT" library="cpio" package="XH-A-3" value="XH-A-3" x="-71.12" y="46.99"/>
 <element name="SENS_TEMP_0" library="cpio" package="XH-A-3" value="XH-A-3" x="-17.78" y="53.34"/>
 <element name="SENS_TEMP_1" library="cpio" package="XH-A-3" value="XH-A-3" x="-27.94" y="53.34"/>
@@
 <contactref element="HEAT_1" pad="2"/>
 <contactref element="R_HSS_GND" pad="2"/>
-<contactref element="SENS_PH1" pad="3"/>
+<contactref element="SENS_BRIGHT" pad="3"/>
 <contactref element="SENS_PH" pad="3"/>
 <contactref element="CAMERA" pad="6"/>
@@
 <contactref element="R_PUSHBUT1" pad="2"/>
 <contactref element="SENS_PH" pad="1"/>
-<contactref element="SENS_PH1" pad="1"/>
+<contactref element="SENS_BRIGHT" pad="1"/>
 <contactref element="C_IO1" pad="1"/>
 <wire x1="-18.15" y1="73.66" x2="-15.61" y2="76.2" width="0" layer="19" extent="1-1"/>
@@
 <signal name="N$35">
 <contactref element="R_BRIGHT" pad="2"/>
-<contactref element="SENS_PH1" pad="2"/>
+<contactref element="SENS_BRIGHT" pad="2"/>
 <wire x1="-71.12" y1="46.99" x2="-44.82" y2="76.2" width="0" layer="19" extent="1-1"/>
 </signal>
