File: cpio-pcb/eagle-proj/cpio/cpio.sch (EAGLE design)
At the start: 76 parts

Commit message: schematic revised and first BOM
Parts:
- removed BEEP: BEEPER, cpio:BEEPER
- removed LED_PWR_12V, LED_PWR_3.3V, LED_PWR_5V, LED_RP: (no value), SparkFun-LED:LED1206
- removed PUSH1: BUTTON, cpio:BUTTON
- removed R_BEP, R_LED_12V, R_LED_5V: (no value), SparkFun-Passives:RESISTOR0805-RES
- removed R_HSS_GND: 1k, SparkFun-Passives:RESISTOR0805-RES
- removed R_HSS_PROT_0, R_HSS_PROT_1, R_HSS_PROT_2, R_HSS_PROT_3, R_HSS_SD: 10k, SparkFun-Passives:RESISTOR0805-RES
- removed SENS_BRIGHT, SENS_PH: XH-A-3, cpio:XH-A-3
- removed U$2: DB2X41100L, cpio:DB2X41100L
- added JP1, JP2: (no value), SparkFun-Connectors:M03PTH
- added LED1, LED2: (no value), led:LEDSML0805
- added S1: (no value), switch-omron:10-XX
- added U$3, U$4, U$5, U$6: SPACERHOLE, cpio:SPACERHOLE
- C_SD_1: value 4.7u -> 10u
- C_SD_3: value 10n -> 100n
- R_BRIGHT, R_LED_3.3V, R_LED_RP, R_PUSHBUT1: value (none) -> 1k
- R_CM_LOAD, R_CM_U0: value 100 -> 10k
- R_CM_SENS: value 1m -> 10m
- R_CM_U1: value 100 -> 1k
- R_PH: value 10k -> 1k
- R_PUSHBUT2: value (none) -> 100
- renumbered R_CM_LOAD1 to R_CM_U0, R_CM_LOAD2 to R_CM_U1
Connections:
- removed net GPIO17: BEEP.-
- removed net N$11: LED_PWR_5V.A, R_LED_5V.1
- removed net N$23: U$2.A
- removed net N$30: R_HSS_SD.1, SWT_HEAT.STAT_DIS
- removed net N$31: R_HSS_PROT_3.2, SWT_HEAT.INPUT4
- removed net N$32: R_HSS_PROT_2.2, SWT_HEAT.INPUT3
- removed net N$33: R_HSS_PROT_1.2, SWT_HEAT.INPUT2
- removed net N$34: R_HSS_PROT_0.2, SWT_HEAT.INPUT1
- removed net N$4: R_HSS_GND.1, SWT_HEAT.GND
- removed net N$5: PUSH1.P$2, R_PUSHBUT2.1
- removed net N$64: BEEP.+, R_BEP.1
- net 12V: no longer R_LED_12V.2
- net 3.3V: now also JP1.1, JP2.1; no longer R_BEP.2, R_HSS_SD.2, SENS_BRIGHT.1, SENS_PH.1
- net 5V: no longer R_LED_5V.2
- net GND: now also JP1.3, JP2.3, LED1.C, LED2.C, S1.P, S1.P1; no longer LED_PWR_12V.C, LED_PWR_3.3V.C, LED_PWR_5V.C, LED_RP.C, PUSH1.P$1, R_HSS_GND.2, SENS_BRIGHT.3, SENS_PH.3
- net GPIO13: now also SWT_HEAT.INPUT1; no longer R_HSS_PROT_0.1
- net GPIO19: now also SWT_HEAT.INPUT2; no longer R_HSS_PROT_1.1
- net GPIO21: now also SWT_HEAT.INPUT4; no longer R_HSS_PROT_3.1
- net GPIO26: now also SWT_HEAT.INPUT3; no longer R_HSS_PROT_2.1
- net N$15: now also LED2.A; no longer LED_PWR_3.3V.A
- net N$2: now also R_PUSHBUT2.1, S1.S, S1.S1; no longer LED_PWR_12V.A, R_LED_12V.1
- net N$20: now also LED1.A; no longer LED_RP.A
- net N$24: no longer U$2.C
- net N$35: now also JP1.2; no longer SENS_BRIGHT.2
- net N$7: now also JP2.2; no longer SENS_PH.2
Other:
- note removed: "Ground Diode missing!"
- note removed: "Load Diode missing!"
- note removed: "Pull UP Required?"
- moved on the sheet: LDO

Commit message: schematic revs...
Parts:
- added R_BRIGHT1, R_BRIGHT2: 1k, SparkFun-Passives:RESISTOR0805-RES
Connections:
- net 3.3V: now also R_BRIGHT2.2
- net ADC_BRIGHT: now also R_BRIGHT1.2
- net GND: now also R_BRIGHT1.1
- net N$35: now also R_BRIGHT2.1
Changed lines of the file:
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@@
 <part name="LED1" library="led" deviceset="LED" device="SML0805"/>
 <part name="LED2" library="led" deviceset="LED" device="SML0805"/>
+<part name="R_BRIGHT1" library="SparkFun-Passives" deviceset="RESISTOR" device="0805-RES" value="1k"/>
+<part name="R_BRIGHT2" library="SparkFun-Passives" deviceset="RESISTOR" device="0805-RES" value="1k"/>
+<part name="SUPPLY12" library="SparkFun-Aesthetics" deviceset="3.3V" device=""/>
+<part name="GND10" library="supply1" deviceset="GND" device=""/>
 </parts>
 <sheets>
@@
 <instance part="LED1" gate="G$1" x="38.1" y="-66.04"/>
 <instance part="LED2" gate="G$1" x="264.16" y="-226.06"/>
+<instance part="R_BRIGHT1" gate="G$1" x="426.72" y="-208.28" rot="R90"/>
+<instance part="R_BRIGHT2" gate="G$1" x="436.88" y="-198.12" rot="R90"/>
+<instance part="SUPPLY12" gate="G$1" x="436.88" y="-193.04"/>
+<instance part="GND10" gate="1" x="426.72" y="-215.9"/>
 </instances>
 <busses>
@@
 <junction x="119.38" y="-147.32"/>
 </segment>
+<segment>
+<pinref part="R_BRIGHT1" gate="G$1" pin="1"/>
+<pinref part="GND10" gate="1" pin="GND"/>
+</segment>
 </net>
 <net name="GPIO17" class="0">
@@
 <pinref part="JP2" gate="G$1" pin="1"/>
 </segment>
+<segment>
+<pinref part="R_BRIGHT2" gate="G$1" pin="2"/>
+<pinref part="SUPPLY12" gate="G$1" pin="3.3V"/>
+</segment>
 </net>
 <net name="N$15" class="0">
@@
 <wire x1="447.04" y1="-203.2" x2="436.88" y2="-203.2" width="0.1524" layer="91"/>
 <pinref part="JP1" gate="G$1" pin="2"/>
+<pinref part="R_BRIGHT2" gate="G$1" pin="1"/>
+<junction x="436.88" y="-203.2"/>
 </segment>
 </net>
@@
 <wire x1="419.1" y1="-203.2" x2="406.4" y2="-203.2" width="0.1524" layer="91"/>
 <junction x="419.1" y="-203.2"/>
-</segment>
-<segment>
+<pinref part="R_BRIGHT1" gate="G$1" pin="2"/>
+<junction x="426.72" y="-203.2"/>
+</segment>
+<segment>
